Commit message: add mobile manipulator

File: aircraft_scanning_description/urdf/quadrotor_camera.urdf.xacro (robot description, xacro)
@@ -1,5 +1,4 @@
 <?xml version="1.0"?>
 <robot name="quadrotor" xmlns:xacro="http://www.ros.org/wiki/xacro">
-    <xacro:property name="M_PI" value="3.1415926535897931" />
     <!--quadrotor_base-->
     <xacro:include filename="$(find hector_quadrotor_description)/urdf/quadrotor_base.urdf.xacro" />
@@ -58,5 +57,7 @@
     <!-- add two links and joints for controlling the depth camera rs435 -->
     <xacro:include filename="$(find aircraft_scanning_description)/urdf/rgbd_camera.urdf.xacro"/>
-    <xacro:quadrotor_camera_macro parent="camera_link"/>
+    <xacro:camera_macro parent="camera_link">
+      <origin xyz="0.035 0 0" rpy="0 0 0"/>
+    </xacro:camera_macro>
     <gazebo reference="base_fixed_link">
       <material>Gazebo/Orange</material>
@@ -83,3 +84,4 @@
       </plugin>
     </gazebo>
+    <xacro:include filename="$(find hector_quadrotor_gazebo)/urdf/quadrotor_plugins.gazebo.xacro" />
 </robot>

File: aircraft_scanning_description/urdf/rgbd_camera.urdf.xacro (robot description, xacro)
@@ -14,7 +14,8 @@
   <xacro:property name="realsense_d435_case_offset_y" value="-0.0175"/>
   <xacro:property name="realsense_d435_case_offset_z" value="0.0"/>
-  <xacro:macro name="quadrotor_camera_macro" params="parent">
+  <xacro:property name="rpy" value="0 0 0"/>
+  <xacro:macro name="camera_macro" params="parent *origin">
     <joint name="rs435_joint" type="fixed">
-      <origin xyz="0.035 0 0" rpy="0 0 0"/>
+      <xacro:insert_block name="origin"/>
       <parent link="${parent}"/>
       <child link="rs435_link"/>
