Commit message: support transformation of mobile to camera

File: aircraft_scanning_description/urdf/4wheel_base.urdf.xacro (robot description, xacro)
@@ -21,5 +21,5 @@
     <xacro:property name="support_x" value="1.0" />
     <xacro:property name="support_y" value="0.8" />
-    <xacro:property name="support_z" value="0.6" />
+    <xacro:property name="support_z" value="0.5" />
     <xacro:property name="support_m" value="30" />
     <!-- main triwheeler link -->
@@ -286,5 +286,5 @@
       </gazebo>
       <gazebo reference="link_fbumper">
-        <material>Gazebo/DarkGrey</material>
+        <material>Gazebo/Yellow</material>
       </gazebo>
       <gazebo reference="link_rbumper">

File: aircraft_scanning_description/urdf/mobile_manipulator.urdf.xacro (robot description, xacro)
@@ -10,10 +10,15 @@
     <xacro:include filename="$(find iiwa_description)/urdf/iiwa14.xacro"/>
     <xacro:iiwa14 hardware_interface="$(arg hardware_interface)" robot_name="iiwa" parent="link_support">
-      <origin xyz="0 0 0.6" rpy="0 0 0" />
+      <origin xyz="0 0 0.5" rpy="0 0 0" />
+      <xacro:property name="safety_controller_k_pos" value="100" />
+      <xacro:property name="safety_controller_k_vel" value="2" />
+      <xacro:property name="joint_damping" value="1" />
+      <xacro:property name="max_effort" value="300"/>
+      <xacro:property name="max_velocity" value="2"/>
     </xacro:iiwa14>
     <!--camera-->
     <xacro:include filename="$(find aircraft_scanning_description)/urdf/rgbd_camera.urdf.xacro"/>
     <xacro:camera_macro parent="iiwa_link_ee">
-        <origin xyz="0 0 0.025" rpy="0 -${PI/2} 0" />
+        <origin xyz="0 0 0.0208" rpy="0 -${PI/2} 0" />
     </xacro:camera_macro>
 </robot>
